File: Board/Board.kicad_pcb (KiCad board)
At the start: 2 copper layers, 55 parts, among them J1 Screw_Terminal_1x02, P1 USB_B, P2 CONN_01X05, P3 CONN_01X06, SW1 SW_SPST, SW2 SW_SPST, U1 MCP23016, U2 LM1117-3.3, U3 MCP9808, U4 ESP-12E

Commit message: Layout rev 1
Parts:
- moved R24 147.1 mm to (139.1, 71.1)
- moved SW1 133.9 mm to (142.9, 99.7), turned to 90 degrees
- moved R25 93.1 mm to (139.1, 73.0)
- moved C8 90.9 mm to (111.1, 102.9)
- moved P3 83.6 mm to (120.7, 95.9)
- moved C10 83.5 mm to (116.2, 102.9)
- moved C9 83.5 mm to (113.7, 102.9)
- moved R30 79.5 mm to (139.1, 77.5)
- moved R26 78.8 mm to (139.1, 88.9)
- moved R27 78.8 mm to (139.1, 85.1), turned to 180 degrees
- moved R28 78.8 mm to (139.1, 87.0)
- moved R29 78.8 mm to (139.1, 81.3)
- moved R31 78.8 mm to (139.1, 83.2)
- moved R19 78.4 mm to (113.7, 80.6)
- moved R20 78.4 mm to (113.7, 78.7)
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Connections:
- C6 pad 1: Net-(C6-Pad1) -> VCC
- P2 pad 1: RX -> TX
- P2 pad 3: TX -> RX
- P3 pad 2: MISO -> CS
- P3 pad 3: MOSI -> MISO
- P3 pad 4: SCK -> MOSI
- P3 pad 5: CS -> SCK
- U3 pad 8: Net-(C6-Pad1) -> VCC
Routing:
- net VCC: track 58.9 -> 174.8 mm, vias 2 -> 8
- net RX: track 0.00 -> 76.5 mm
- net TX: track 0.00 -> 72.6 mm
- net SDA: track 0.00 -> 69.4 mm, vias 0 -> 3
- net SCL: track 0.00 -> 66.2 mm, vias 0 -> 3
- net IOINT: track 0.00 -> 41.0 mm, vias 0 -> 4
- net Net-(R24-Pad2): track 0.00 -> 33.4 mm, vias 0 -> 2
- net RESET: track 0.00 -> 32.0 mm
- net Alert: track 0.00 -> 25.7 mm, vias 0 -> 2
- net Net-(R25-Pad2): track 0.00 -> 25.0 mm, vias 0 -> 2
- net GND: track 6.10 -> 30.1 mm, vias 0 -> 2
- net PROG: track 0.00 -> 21.6 mm
- net STATUS: track 0.00 -> 20.3 mm, vias 0 -> 2
- net VDD: track 32.4 -> 46.6 mm
- net MISO: track 0.00 -> 6.18 mm
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Other:
- board outline added: 69.9 x 58.4 mm

Commit message: Final Rev 1
Parts:
- removed C10: 22µ, Capacitors_SMD:C_1206_HandSoldering
- added REF**: MountingHole_2.2mm_M2_ISO7380, Mounting_Holes:MountingHole_2.2mm_M2_ISO7380, F.Cu at (92.1, 87.6)
- added REF**: MountingHole_2.2mm_M2_ISO7380, Mounting_Holes:MountingHole_2.2mm_M2_ISO7380, F.Cu at (143.5, 66.7)
- added REF**: MountingHole_2.2mm_M2_ISO7380, Mounting_Holes:MountingHole_2.2mm_M2_ISO7380, F.Cu at (107.3, 110.5)
- C7: value 100n -> 22µ; footprint Capacitors_SMD:C_0603_HandSoldering -> Capacitors_SMD:C_1206_HandSoldering
- moved C7 16.3 mm to (111.1, 102.9), turned to 270 degrees
- moved C8 2.54 mm to (113.7, 102.9)
- moved C9 2.54 mm to (116.2, 102.9)
Connections:
- D3 pad 1: (no net) -> Net-(D3-Pad1)
- D3 pad 4: (no net) -> Net-(D3-Pad4)
- P1 pad 2: (no net) -> Net-(P1-Pad2)
- P1 pad 3: (no net) -> Net-(P1-Pad3)
- P1 pad 5: (no net) -> Net-(P1-Pad5)
- U1 pad 10: (no net) -> GND
- U4 pad 19: (no net) -> Net-(U4-Pad19)
- U4 pad 2: (no net) -> Net-(U4-Pad2)
- U4 pad 20: (no net) -> Net-(U4-Pad20)
Routing:
- net VCC: track 174.8 -> 197.4 mm, vias 8 -> 9
- net VDD: track 46.6 -> 61.9 mm
- net GND: track 30.1 -> 24.0 mm
- net Net-(R2-Pad2): track 44.1 -> 45.2 mm
- net Net-(R3-Pad2): track 44.9 -> 45.6 mm
- added copper zone on B.Cu, net GND
- added copper zone on F.Cu, net GND
Other:
- outline, holes or cut-outs redrawn
- net class PWR: clearance 0.2032 -> 0.1524
- rule trace_min: 0.2 -> 0.1524
- rule via_min_size: 0.4 -> 0.3302
- board text added: "CS"
- board text added: "CloudTempSensor rev. 1"
- board text added: "GND"
- board text added: "MISO"
- board text added: "MOSI"
- board text added: "PRG"
- board text added: "RST"
- board text added: "RX"
- board text added: "SCK"
- board text added: "TX"
- board text added: "VCC"
- board text added: "VCC = 3,3V VDD min. 5V max. 20V VDD connected to USB power!"
- board text added: "VDD"
- board text added: "https://github.com/penguineer/CloudTempSensor"
