File: Board/Board.kicad_pcb (KiCad board)
At the start: 2 copper layers, 69.9 x 58.4 mm, 56 parts, among them J1 Screw_Terminal_1x02, P1 USB_B, P2 CONN_01X05, P3 CONN_01X06, P4 CONN_01X03, SW1 SW_SPST, SW2 SW_SPST, U1 MCP23016, U2 LM1117-3.3, U3 MCP9808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

Commit message: Minor changes for rev3
Parts:
- added R33: 0, Resistors_SMD:R_0603_HandSoldering, F.Cu at (124.5, 113.7)
- moved P1 1.27 mm to (128.3, 114.9)
Routing:
- net Net-(P1-Pad5): track 0.00 -> 2.71 mm
- net VDD: track 54.1 -> 55.7 mm
Other:
- outline, holes or cut-outs redrawn
Changed lines of the file:
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@@
 (kicad_pcb (version 4) (host pcbnew 4.0.5+dfsg1-4)
   (general
-    (links 124)
+    (links 126)
     (no_connects 0)
-    (area 76.759999 63.424999 146.760001 121.995001)
+    (area 76.759999 62.5476 153.019543 122.3674)
     (thickness 1.6)
     (drawings 33)
-    (tracks 412)
+    (tracks 417)
     (zones 0)
-    (modules 56)
+    (modules 57)
     (nets 67)
   )
@@
       (linewidth 0.100000)
       (plotframeref false)
-      (viasonmask false)
+      (viasonmask true)
       (mode 1)
       (useauxorigin false)
@@
   )
   (module Connect:USB_Micro-B (layer F.Cu)
-    (at 127 114.935 90)
+    (at 128.27 114.935 90)
     (descr "Micro USB Type B Receptacle")
     (tags "USB USB_B USB_micro USB_OTG")
@@
     )
   )
+  (module Resistors_SMD:R_0603_HandSoldering (layer F.Cu)
+    (at 124.46 113.665 90)
+    (descr "Resistor SMD 0603, hand soldering")
+    (tags "resistor 0603")
+    (attr smd)
+    (fp_text reference R33 (at 0 -1.9 90) (layer F.SilkS)
+      (effects (font (size 1 1) (thickness 0.15)))
+    )
+    (fp_text value 0 (at 0 1.9 90) (layer F.Fab)
+      (effects (font (size 1 1) (thickness 0.15)))
+    )
+    (fp_line (start -0.8 0.4) (end -0.8 -0.4) (layer F.Fab) (width 0.1))
+    (fp_line (start 0.8 0.4) (end -0.8 0.4) (layer F.Fab) (width 0.1))
+    (fp_line (start 0.8 -0.4) (end 0.8 0.4) (layer F.Fab) (width 0.1))
+    (fp_line (start -0.8 -0.4) (end 0.8 -0.4) (layer F.Fab) (width 0.1))
+    (fp_line (start -2 -0.8) (end 2 -0.8) (layer F.CrtYd) (width 0.05))
+    (fp_line (start -2 0.8) (end 2 0.8) (layer F.CrtYd) (width 0.05))
+    (fp_line (start -2 -0.8) (end -2 0.8) (layer F.CrtYd) (width 0.05))
+    (fp_line (start 2 -0.8) (end 2 0.8) (layer F.CrtYd) (width 0.05))
+    (fp_line (start 0.5 0.675) (end -0.5 0.675) (layer F.SilkS) (width 0.15))
+    (fp_line (start -0.5 -0.675) (end 0.5 -0.675) (layer F.SilkS) (width 0.15))
+    (pad 1 smd rect (at -1.1 0 90) (size 1.2 0.9) (layers F.Cu F.Paste F.Mask)
+      (net 2 GND))
+    (pad 2 smd rect (at 1.1 0 90) (size 1.2 0.9) (layers F.Cu F.Paste F.Mask)
+      (net 63 "Net-(P1-Pad5)"))
+    (model Resistors_SMD.3dshapes/R_0603_HandSoldering.wrl
+      (at (xyz 0 0 0))
+      (scale (xyz 1 1 1))
+      (rotate (xyz 0 0 0))
+    )
+  )
+  (gr_line (start 132.715 106.045) (end 145.415 106.045) (angle 90) (layer Edge.Cuts) (width 0.15))
+  (gr_line (start 131.445 120.65) (end 131.445 107.315) (angle 90) (layer Edge.Cuts) (width 0.15))
+  (gr_line (start 78.105 121.92) (end 130.175 121.92) (angle 90) (layer Edge.Cuts) (width 0.15))
+  (gr_line (start 146.685 104.775) (end 146.685 64.77) (angle 90) (layer Edge.Cuts) (width 0.15))
   (gr_text SDA (at 109.855 100.965) (layer F.SilkS)
     (effects (font (size 1 1) (thickness 0.1)) (justify left))
@@
     (effects (font (size 1 1) (thickness 0.1)) (justify left))
   )
-  (gr_line (start 146.685 107.315) (end 146.685 64.77) (angle 90) (layer Edge.Cuts) (width 0.15))
-  (gr_line (start 132.08 108.585) (end 145.415 108.585) (angle 90) (layer Edge.Cuts) (width 0.15))
-  (gr_line (start 130.81 120.65) (end 130.81 109.855) (angle 90) (layer Edge.Cuts) (width 0.15))
-  (gr_line (start 78.105 121.92) (end 129.54 121.92) (angle 90) (layer Edge.Cuts) (width 0.15))
-  (gr_arc (start 132.08 109.855) (end 130.81 109.855) (angle 90) (layer Edge.Cuts) (width 0.15))
-  (gr_arc (start 129.54 120.65) (end 130.81 120.65) (angle 90) (layer Edge.Cuts) (width 0.15))
-  (gr_arc (start 145.415 107.315) (end 146.685 107.315) (angle 90) (layer Edge.Cuts) (width 0.15))
+  (gr_arc (start 132.715 107.315) (end 131.445 107.315) (angle 90) (layer Edge.Cuts) (width 0.15))
+  (gr_arc (start 130.175 120.65) (end 131.445 120.65) (angle 90) (layer Edge.Cuts) (width 0.15))
+  (gr_arc (start 145.415 104.775) (end 146.685 104.775) (angle 90) (layer Edge.Cuts) (width 0.15))
   (gr_line (start 76.835 64.77) (end 76.835 120.65) (angle 90) (layer Edge.Cuts) (width 0.15))
   (gr_line (start 145.415 63.5) (end 78.105 63.5) (angle 90) (layer Edge.Cuts) (width 0.15))
@@
   (segment (start 101.77 98.575) (end 101.92 98.425) (width 0.2032) (layer F.Cu) (net 3))
   (segment (start 99.441 100.33) (end 101.77 100.33) (width 0.2032) (layer F.Cu) (net 3))
-  (segment (start 118.745 114.3) (end 119.38 114.3) (width 0.4064) (layer F.Cu) (net 4))
-  (segment (start 119.38 114.3) (end 121.3159 116.2359) (width 0.4064) (layer F.Cu) (net 4))
-  (segment (start 121.3159 116.2359) (end 125.43746 116.2359) (width 0.4064) (layer F.Cu) (net 4))
+  (segment (start 126.70746 116.2359) (end 125.1259 116.2359) (width 0.4064) (layer F.Cu) (net 4))
+  (segment (start 118.745 114.3) (end 119.38 114.3) (width 0.4064) (layer F.Cu) (net 4) (status 30))
+  (segment (start 119.38 114.3) (end 121.3159 116.2359) (width 0.4064) (layer F.Cu) (net 4) (status 10))
+  (segment (start 121.3159 116.2359) (end 125.1259 116.2359) (width 0.4064) (layer F.Cu) (net 4))
+  (segment (start 125.1259 116.2359) (end 125.43746 116.2359) (width 0.4064) (layer F.Cu) (net 4))
   (segment (start 82.55 118.745) (end 114.3 118.745) (width 0.4064) (layer B.Cu) (net 4))
-  (segment (start 114.3 118.745) (end 118.745 114.3) (width 0.4064) (layer B.Cu) (net 4))
+  (segment (start 114.3 118.745) (end 118.745 114.3) (width 0.4064) (layer B.Cu) (net 4) (status 20))
   (segment (start 86.995 118.84) (end 82.645 118.84) (width 0.4064) (layer F.Cu) (net 4))
   (segment (start 82.645 118.84) (end 82.55 118.745) (width 0.4064) (layer F.Cu) (net 4))
@@
   (segment (start 135.7 78.93) (end 133.38 78.93) (width 0.2032) (layer F.Cu) (net 58))
   (segment (start 137.16 77.47) (end 135.7 78.93) (width 0.2032) (layer F.Cu) (net 58))
+  (segment (start 126.70746 113.6359) (end 125.5051 113.6359) (width 0.2032) (layer F.Cu) (net 63))
+  (segment (start 125.5051 113.6359) (end 124.46 112.5908) (width 0.2032) (layer F.Cu) (net 63))
+  (segment (start 124.46 112.5908) (end 124.46 112.565) (width 0.2032) (layer F.Cu) (net 63))
   (zone (net 0) (net_name "") (layer F.Cu) (hatch edge 0.508)
     (connect_pads (clearance 0.254))
@@
     (polygon
       (pts
-        (xy 146.685 108.585) (xy 130.81 108.585) (xy 130.81 121.92) (xy 76.835 121.92) (xy 76.835 63.5)
+        (xy 146.685 106.045) (xy 131.445 106.045) (xy 131.445 121.92) (xy 76.835 121.92) (xy 76.835 63.5)
         (xy 146.685 63.5)
       )
@@
     (polygon
       (pts
-        (xy 146.685 108.585) (xy 130.81 108.585) (xy 130.81 121.92) (xy 76.835 121.92) (xy 76.835 63.5)
+        (xy 146.685 106.045) (xy 131.445 106.045) (xy 131.445 121.92) (xy 76.835 121.92) (xy 76.835 63.5)
         (xy 146.685 63.5)
       )
@@
     (polygon
       (pts
-        (xy 116.205 89.535) (xy 114.935 89.535) (xy 114.935 66.04) (xy 116.205 66.04)
+        (xy 116.84 89.535) (xy 116.205 89.535) (xy 116.205 72.39) (xy 116.84 72.39)
       )
     )
@@
     (polygon
       (pts
-        (xy 116.205 89.535) (xy 114.935 89.535) (xy 114.935 66.04) (xy 116.205 66.04)
+        (xy 116.84 89.535) (xy 116.205 89.535) (xy 116.205 72.39) (xy 116.84 72.39)
       )
     )
@@
     (polygon
       (pts
-        (xy 116.205 102.87) (xy 116.205 120.015) (xy 114.935 120.015) (xy 114.935 102.87)
+        (xy 116.84 102.87) (xy 116.84 120.015) (xy 116.205 120.015) (xy 116.205 102.87)
       )
     )
@@
     (polygon
       (pts
-        (xy 116.205 102.87) (xy 116.205 120.015) (xy 114.935 120.015) (xy 114.935 102.87)
+        (xy 116.84 102.87) (xy 116.84 120.015) (xy 116.205 120.015) (xy 116.205 102.87)
       )
     )
